File: Blinky.sch (KiCad schematic (older format))
At the start: 7 parts, among them U1 7555

Commit message: Fix capacitor footprint - should have been 0805
Parts:
- C1: footprint Capacitors_SMD:C_1206_HandSoldering -> Capacitors_SMD:C_0805_HandSoldering
Changed lines of the file:
@@
 F 0 "C1" H 4925 4700 50  0000 L CNN
 F 1 "1U" H 4925 4500 50  0000 L CNN
-F 2 "Capacitors_SMD:C_1206_HandSoldering" H 4938 4450 50  0001 C CNN
+F 2 "Capacitors_SMD:C_0805_HandSoldering" H 4938 4450 0   0001 C CNN
 F 3 "" H 4900 4600 50  0000 C CNN
 	1    4900 4600
